File: 2024_LED_Breakout_Board/2024_LED_Breakout_Board.kicad_pcb (KiCad board)
At the start: 2 copper layers, 75 x 138 mm, 87 parts, among them J1 43045-1015, J2 43045-1615, J3 43045-2215

Commit message: A few minor fixes
Routing:
- net GND: track 0.00 -> 2.87 mm, vias 0 -> 1
Changed lines of the file:
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@@
 		(tags "Connector")
 		(property "Reference" "J2"
-			(at 0 0 180)
+			(at -16.4856 -5.7 180)
 			(layer "B.SilkS")
 			(effects
@@
 		(tags "Connector")
 		(property "Reference" "J1"
-			(at 0 0 180)
+			(at -12.2036 -3.0572 180)
 			(layer "B.SilkS")
 			(effects
@@
 		(tags "Connector")
 		(property "Reference" "J3"
-			(at 0 0.2 180)
+			(at -21.2288 -1.1992 180)
 			(layer "B.SilkS")
 			(effects
@@
 		)
 	)
-	(gr_rect
-		(start 127 155.5)
-		(end 184.5 166.5)
-		(stroke
-			(width 0.2)
-			(type default)
-		)
-		(fill none)
-		(layer "F.Cu")
-	)
-	(gr_rect
-		(start 131 88.5)
-		(end 170.5 102.5)
-		(stroke
-			(width 0.2)
-			(type default)
-		)
-		(fill none)
-		(layer "F.Cu")
-	)
-	(gr_rect
-		(start 128 123)
-		(end 192.5 136.5)
-		(stroke
-			(width 0.2)
-			(type default)
-		)
-		(fill none)
-		(layer "F.Cu")
-	)
-	(gr_rect
-		(start 127 182)
-		(end 197 191.5)
-		(stroke
-			(width 0.2)
-			(type default)
-		)
-		(fill none)
-		(layer "F.Cu")
-	)
 	(gr_line
 		(start 193.6 196)
@@
 		(layer "Edge.Cuts")
 	)
-	(gr_text "Power Outputs"
-		(at 173.5 95.5 0)
-		(layer "F.Cu")
-		(effects
-			(font
-				(size 1.5 1.5)
-				(thickness 0.3)
-				(bold yes)
-			)
-			(justify left bottom)
-		)
-	)
-	(gr_text "Safety Circuit"
-		(at 153 195 0)
-		(layer "F.Cu")
-		(effects
-			(font
-				(size 1.5 1.5)
-				(thickness 0.3)
-				(bold yes)
-			)
-			(justify left bottom)
-		)
-	)
-	(gr_text "AIR Path"
-		(at 187 162 0)
-		(layer "F.Cu")
-		(effects
-			(font
-				(size 1.5 1.5)
-				(thickness 0.3)
-				(bold yes)
-			)
-			(justify left bottom)
-		)
-	)
-	(gr_text "BSPD Logic"
-		(at 183 140.5 0)
-		(layer "F.Cu")
-		(effects
-			(font
-				(size 1.5 1.5)
-				(thickness 0.3)
-				(bold yes)
-			)
-			(justify left bottom)
-		)
-	)
 	(gr_text "BRAKE_LIGHT_SIG"
 		(at 166.925 88.2 90)
@@
 		)
 	)
+	(gr_text "Power Outputs"
+		(at 128.016 134.0612 90)
+		(layer "F.SilkS")
+		(effects
+			(font
+				(size 1.5 1.5)
+				(thickness 0.3)
+				(bold yes)
+			)
+			(justify left bottom)
+		)
+	)
+	(gr_text "Safety Circuit"
+		(at 127.3556 191.3128 90)
+		(layer "F.SilkS")
+		(effects
+			(font
+				(size 1.5 1.5)
+				(thickness 0.3)
+				(bold yes)
+			)
+			(justify left bottom)
+		)
+	)
+	(gr_text "AIR Path"
+		(at 127.7112 164.5412 90)
+		(layer "F.SilkS")
+		(effects
+			(font
+				(size 1.5 1.5)
+				(thickness 0.3)
+				(bold yes)
+			)
+			(justify left bottom)
+		)
+	)
+	(gr_text "BSPD Logic"
+		(at 128.7272 97.9424 90)
+		(layer "F.SilkS")
+		(effects
+			(font
+				(size 1.5 1.5)
+				(thickness 0.3)
+				(bold yes)
+			)
+			(justify left bottom)
+		)
+	)
+	(dimension
+		(type aligned)
+		(layer "Dwgs.User")
+		(pts
+			(xy 193.6 70) (xy 193.5 196)
+		)
+		(height -18.046679)
+		(gr_text "126.0000 mm"
+			(at 210.446673 133.01341 89.95452717)
+			(layer "Dwgs.User")
+			(effects
+				(font
+					(size 1 1)
+					(thickness 0.15)
+				)
+			)
+		)
+		(format
+			(prefix "")
+			(suffix "")
+			(units 3)
+			(units_format 1)
+			(precision 4)
+		)
+		(style
+			(thickness 0.1)
+			(arrow_length 1.27)
+			(text_position_mode 0)
+			(extension_height 0.58642)
+			(extension_offset 0.5) keep_text_aligned)
+	)
+	(dimension
+		(type aligned)
+		(layer "Dwgs.User")
+		(pts
+			(xy 130.6 70) (xy 193.6 70)
+		)
+		(height -11.6816)
+		(gr_text "63.0000 mm"
+			(at 162.1 57.1684 0)
+			(layer "Dwgs.User")
+			(effects
+				(font
+					(size 1 1)
+					(thickness 0.15)
+				)
+			)
+		)
+		(format
+			(prefix "")
+			(suffix "")
+			(units 3)
+			(units_format 1)
+			(precision 4)
+		)
+		(style
+			(thickness 0.1)
+			(arrow_length 1.27)
+			(text_position_mode 0)
+			(extension_height 0.58642)
+			(extension_offset 0.5) keep_text_aligned)
+	)
 	(segment
 		(start 153 101.5)
@@
 	)
 	(segment
+		(start 191.05 184.4)
+		(end 191.05 181.9744)
+		(width 0.2)
+		(layer "F.Cu")
+		(net 2)
+	)
+	(segment
+		(start 191.05 181.9744)
+		(end 191.3636 181.6608)
+		(width 0.2)
+		(layer "F.Cu")
+		(net 2)
+	)
+	(via
+		(at 191.3636 181.6608)
+		(size 0.6)
+		(drill 0.3)
+		(layers "F.Cu" "B.Cu")
+		(net 2)
+	)
+	(segment
 		(start 156.55 95)
 		(end 156.55 97.025)
@@
 	)
 	(segment
-		(start 172.575 164.025)
+		(start 172.575 164.5846)
 		(end 172.575 162)
 		(width 0.2)
@@
 	)
 	(segment
-		(start 171.55 165.05)
-		(end 172.575 164.025)
+		(start 170.18 166.9796)
+		(end 172.575 164.5846)
 		(width 0.2)
 		(layer "F.Cu")
@@
 	)
 	(via
-		(at 171.55 165.05)
+		(at 170.18 166.9796)
 		(size 0.6)
 		(drill 0.3)
@@
 	)
 	(segment
-		(start 159.62 167.07)
-		(end 158.05 165.5)
+		(start 170.18 166.9796)
+		(end 170.0896 167.07)
 		(width 0.2)
 		(layer "B.Cu")
@@
 	)
 	(segment
-		(start 169.53 167.07)
-		(end 159.62 167.07)
+		(start 159.62 167.07)
+		(end 158.05 165.5)
 		(width 0.2)
 		(layer "B.Cu")
@@
 	)
 	(segment
-		(start 171.55 165.05)
-		(end 169.53 167.07)
+		(start 170.0896 167.07)
+		(end 159.62 167.07)
 		(width 0.2)
 		(layer "B.Cu")

Commit message: Further changes added
Routing:
- net GND: track 2.87 -> 127.5 mm, vias 1 -> 40
- net Net-(LED6-A): track 11.1 -> 4.00 mm, vias 1 -> 0
- net Net-(LED10-A): track 10.9 -> 4.00 mm, vias 1 -> 0
- net Net-(LED11-A): track 10.6 -> 4.00 mm, vias 1 -> 0
- net Net-(LED14-A): track 10.4 -> 4.00 mm, vias 1 -> 0
- net Net-(LED15-A): track 10.4 -> 4.00 mm, vias 1 -> 0
- net Net-(LED20-A): track 10.3 -> 4.00 mm, vias 1 -> 0
- net Net-(LED19-A): track 10.3 -> 4.00 mm, vias 1 -> 0
- net Net-(LED18-A): track 10.3 -> 4.00 mm, vias 1 -> 0
- net Net-(LED17-A): track 10.3 -> 4.00 mm, vias 1 -> 0
- net Net-(LED16-A): track 10.2 -> 4.00 mm, vias 1 -> 0
- net Net-(LED13-A): track 9.97 -> 4.00 mm, vias 1 -> 0
- net Net-(LED12-A): track 9.97 -> 4.00 mm, vias 1 -> 0
- net Net-(LED7-A): track 8.66 -> 4.00 mm, vias 1 -> 0
- net Net-(LED8-A): track 8.46 -> 4.00 mm, vias 1 -> 0
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